File: KiCAD/USB_PD_PSU/USB_PD_PSU.sch (KiCad schematic (older format))
At the start: 4 parts

Commit message: updated schematic and pcb
Changed lines of the file:
@@
 encoding utf-8
 Sheet 1 4
-Title ""
-Date ""
-Rev ""
-Comp ""
+Title "USB PD PSU"
+Date "2020-09-18"
+Rev "1.0"
+Comp "arduonics.com"
 Comment1 ""
 Comment2 ""
@@
 $EndSheet
 Wire Wire Line
-	1750 1800 2200 1800
+	1750 1800 2000 1800
 Wire Wire Line
 	2200 1800 2200 1700
@@
 F0 "LinReg" 50
 F1 "LinReg.sch" 50
-F2 "V_OUT" O R 7050 1400 50
-F3 "GND" B L 4550 2300 50
-F4 "V_IN_BUCK" I L 4550 1900 50
-F5 "V_SNK_IN" I L 4550 1300 50
+F2 "GND" B L 4550 2300 50
+F3 "V_IN_BUCK" I L 4550 1900 50
+F4 "V_SNK_IN" I L 4550 1300 50
+F5 "V_OUT" O R 7050 1400 50
 $EndSheet
 Wire Wire Line
@@
 	1    0    0    -1
 $EndComp
+Wire Wire Line
+	2500 1900 2050 1900
+Wire Wire Line
+	2050 1900 2050 800
+Wire Wire Line
+	2050 800  7350 800
+Wire Wire Line
+	7350 800  7350 1400
+Wire Wire Line
+	7350 1400 7050 1400
+Wire Wire Line
+	2500 2100 2000 2100
+Wire Wire Line
+	2000 2100 2000 1800
+Connection ~ 2000 1800
+Wire Wire Line
+	2000 1800 2200 1800
 $EndSCHEMATC
