File: KiCAD/USB_PD_PSU/LinReg.sch (KiCad schematic (older format))
At the start: 104 parts, among them J3 Conn_02x05_Counter_Clockwise_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, J4 V_OUT_-, J5 V_OUT_+, J6 Conn_02x03_Counter_Clockwise, Q2 BC846BLT1G, Q3 MMBT3906, Q4 FMMT493TA, U10 BCV62CE6327HTSA1, U11 BCV62CE6327HTSA1, U12 LT3081ER-PBF, U13 LT3081ER-PBF, U14 LTC3632, U15 LT3092xST, U5 MCP4822, U6 MCP6422T-E/SN, U7 L78L05_SO8, U8 MCP3202, U9 LT1013DDR

Commit message: updated schematic and pcb
Connections:
- net GND: no longer R45.2
Changed lines of the file:
@@
 encoding utf-8
 Sheet 4 4
-Title ""
-Date ""
-Rev ""
-Comp ""
+Title "USB PD PSU"
+Date "2020-09-18"
+Rev "1.0"
+Comp "arduonics.com"
 Comment1 ""
 Comment2 ""
@@
 	9800 3200 9950 3200
 Wire Wire Line
-	10900 1400 10600 1400
+	10900 1400 10750 1400
 Wire Wire Line
 	9100 1400 9150 1400
@@
 Connection ~ 9100 5400
 Wire Wire Line
-	9100 5050 9100 5000
-Wire Wire Line
-	9100 5000 8800 5000
-Wire Wire Line
 	8500 5000 8250 5000
 Wire Wire Line
@@
 $EndComp
 Wire Wire Line
-	9100 5000 9450 5000
-Wire Wire Line
 	9900 5000 9900 5150
-Connection ~ 9100 5000
 Wire Wire Line
 	9450 5000 9450 5200
@@
 Wire Wire Line
 	5300 7150 5550 7150
+Wire Wire Line
+	8800 5000 9450 5000
+Text HLabel 10750 1200 1    50   Output ~ 0
+V_OUT
+Wire Wire Line
+	10750 1200 10750 1400
+Connection ~ 10750 1400
+Wire Wire Line
+	10750 1400 10600 1400
 $EndSCHEMATC

Commit message: updated KiCad files, added Ibom
Connections:
- net GND: now also R45.2
Changed lines of the file:
@@
 	5300 7150 5550 7150
 Wire Wire Line
-	8800 5000 9450 5000
+	8800 5000 9100 5000
 Text HLabel 10750 1200 1    50   Output ~ 0
 V_OUT
@@
 Wire Wire Line
 	10750 1400 10600 1400
+Wire Wire Line
+	9100 5050 9100 5000
+Connection ~ 9100 5000
+Wire Wire Line
+	9100 5000 9450 5000
 $EndSCHEMATC
