File: KiCAD/USB_PD_PSU/USB_PD_PSU.kicad_pcb (KiCad board)
At the start: 2 copper layers, 161.5 x 57.4 mm, 174 parts, among them J1 USB4105-GF-A, J2 Conn_02x06_Counter_Clockwise, J3 Conn_02x05_Counter_Clockwise_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, J4 V_OUT_-, J5 V_OUT_+, J6 Conn_02x03_Counter_Clockwise, Q1 MMBT3906, Q2 BC846BLT1G, Q3 MMBT3906, Q4 FMMT493TA, U1 STUSB4500QTR, U10 BCV62CE6327HTSA1, U11 BCV62CE6327HTSA1, U12 LT3081ER-PBF, U13 LT3081ER-PBF, U14 LTC3632, U15 LT3092xST, U2 STL6P3LLH6, U3 STL6P3LLH6, U4 SIC438AED, U5 MCP4822, U6 MCP6422T-E/SN, U7 L78L05_SO8, U8 MCP3202, U9 LT1013DDR

Commit message: updated schematic and pcb
Parts:
- moved R18 0.22 mm to (85.3, 49.8)
Connections:
- C15 pad 1: /Buck_Converter/V_OUTPUT -> V_OUTPUT
- R22 pad 1: /Buck_Converter/V_OUTPUT -> V_OUTPUT
- R23 pad 1: /Buck_Converter/V_OUTPUT -> V_OUTPUT
- R45 pad 2: GND -> (no net)
- U4 pad 19: (no net) -> VSNK
Routing:
- net V_OUTPUT: track 75.1 -> 151.5 mm, vias 43 -> 44
- net VSNK: track 185.9 -> 193.2 mm, vias 6 -> 8
- net /Buck_Converter/V_OUTPUT: track 4.83 -> 0.00 mm
- net /LinReg/V_IN_BUCK: track 136.4 -> 137.4 mm
- net GND: track 557.4 -> 557.0 mm, vias 549 -> 547

Commit message: updated KiCad files, added Ibom
Connections:
- R45 pad 2: (no net) -> GND
Routing:
- net VSNK: track 193.2 -> 190.4 mm
- net GND: track 557.0 -> 559.5 mm
